File: HERMES PCB/HERMES PCB.kicad_pcb (KiCad board)
At the start: 2 copper layers, 99.3 x 118.4 mm, 70 parts, among them J1 Conn_01x04, SW1 Rotary_Encoder_Switch, SW2 Rotary_Encoder_Switch, SW3 SW_Push

Commit message: Correction
Parts:
- added G***: LOGO, Logos:NEWblack_logo_Fserif, B.Cu at (91.7, 136.5)
- added G***: LOGO, Logos:NEWblack_logo_Fserif, F.Cu at (92.1, 136.5)
- added G***: LOGO, Logos:NEWblack_logo_soldermask, B.Cu at (91.7, 136.5)
- added G***: LOGO, Logos:NEWblack_logo_soldermask, F.Cu at (92.1, 136.5)

Commit message: Added logos and tested conections
Parts:
- removed REF**: MountingHole_2.2mm_M2, MountingHole:MountingHole_2.2mm_M2
- added 7: MountingHole_2.2mm_M2, MountingHole:MountingHole_2.2mm_M2, F.Cu at (53.2, 156.8)
- added G***: LOGO, NEWblack:Hermes_sandals_Fserif, B.Cu at (145.3, 154.0)
- added G***: LOGO, NEWblack:Hermes_logo-s, F.Cu at (91.8, 153.0)
- added G***: LOGO, NEWblack:Hermes_logo_Fserif_s, B.Cu at (91.9, 153.0)
- added G***: LOGO, NEWblack:Hermes_logo_Fserif_s, F.Cu at (91.8, 153.0)
- added G***: LOGO, NEWblack:Hermes_sandals, F.Cu at (137.3, 54.8)
- added G***: LOGO, NEWblack:Hermes_sandals, F.Cu at (56.4, 153.2)
- added G***: LOGO, NEWblack:Hermes_sandals_Fserif, F.Cu at (137.3, 54.8)
- added G***: LOGO, NEWblack:Hermes_sandals_Fserif, F.Cu at (56.4, 153.2)
- added G***: LOGO, NEWblack:Hermes_sandals_Fcu, F.Cu at (137.3, 54.8)
- added G***: LOGO, NEWblack:Hermes_sandals_Fcu, F.Cu at (56.4, 153.2)
- added G***: LOGO, NEWblack:Hermes_logo_Fcu_s, F.Cu at (91.8, 153.0)
- added G***: LOGO, NEWblack:Hermes_logo-s, B.Cu at (91.9, 153.0)
- D1, D10, D11, D12, D13, D14, D15, D16, D17, D18, D19, D2, D20, D21, D22, D23, D3, D4, D5, D6, D7, D8, D9: footprint Diode_THT:D_DO-35_SOD27_P7.62mm_Horizontal -> NEWblack:D_DO-35_SOD27_P7.62mm_Horizontal
- PRO MICRO BOARD: renamed from B1
- RESET: renamed from SW3; value SW_Push -> RESET
- renumbered REF** to 1, C4 to 100nF, C3 to 100nF, C2 to 100nF, C1 to 100nF, R1 to 10k, REF** to 2, REF** to 3, REF** to 4, REF** to 5, REF** to 6, J1 to OLED, SW1 to RE1, SW2 to RE2
Routing:
- added copper zone on B.Cu, net (none)
