File: HERMES PCB/HERMES PCB.sch (KiCad schematic (older format))
At the start: 61 parts, among them J1 Conn_01x04, SW1 Rotary_Encoder_Switch, SW2 Rotary_Encoder_Switch, SW3 SW_Push

Commit message: Added logos and tested conections
Parts:
- D1, D10, D11, D12, D13, D14, D15, D16, D17, D18, D19, D2, D20, D21, D22, D23, D3, D4, D5, D6, D7, D8, D9: footprint Diode_THT:D_DO-35_SOD27_P7.62mm_Horizontal -> NEWblack:D_DO-35_SOD27_P7.62mm_Horizontal
- SW3: value SW_Push -> RESET
Changed lines of the file:
@@
 F 0 "D1" V 6146 1580 50  0000 R CNN
 F 1 "D_Small" V 6055 1580 50  0000 R CNN
-F 2 "Diode_THT:D_DO-35_SOD27_P7.62mm_Horizontal" V 6100 1650 50  0001 C CNN
+F 2 "NEWblack:D_DO-35_SOD27_P7.62mm_Horizontal" V 6100 1650 50  0001 C CNN
 F 3 "~" V 6100 1650 50  0001 C CNN
 	1    6100 1650
@@
 F 0 "D2" V 6846 1580 50  0000 R CNN
 F 1 "D_Small" V 6755 1580 50  0000 R CNN
-F 2 "Diode_THT:D_DO-35_SOD27_P7.62mm_Horizontal" V 6800 1650 50  0001 C CNN
+F 2 "NEWblack:D_DO-35_SOD27_P7.62mm_Horizontal" V 6800 1650 50  0001 C CNN
 F 3 "~" V 6800 1650 50  0001 C CNN
 	1    6800 1650
@@
 F 0 "D3" V 7346 1580 50  0000 R CNN
 F 1 "D_Small" V 7255 1580 50  0000 R CNN
-F 2 "Diode_THT:D_DO-35_SOD27_P7.62mm_Horizontal" V 7300 1650 50  0001 C CNN
+F 2 "NEWblack:D_DO-35_SOD27_P7.62mm_Horizontal" V 7300 1650 50  0001 C CNN
 F 3 "~" V 7300 1650 50  0001 C CNN
 	1    7300 1650
@@
 F 0 "D4" V 7796 1580 50  0000 R CNN
 F 1 "D_Small" V 7705 1580 50  0000 R CNN
-F 2 "Diode_THT:D_DO-35_SOD27_P7.62mm_Horizontal" V 7750 1650 50  0001 C CNN
+F 2 "NEWblack:D_DO-35_SOD27_P7.62mm_Horizontal" V 7750 1650 50  0001 C CNN
 F 3 "~" V 7750 1650 50  0001 C CNN
 	1    7750 1650
@@
 F 0 "D5" V 6146 2330 50  0000 R CNN
 F 1 "D_Small" V 6055 2330 50  0000 R CNN
-F 2 "Diode_THT:D_DO-35_SOD27_P7.62mm_Horizontal" V 6100 2400 50  0001 C CNN
+F 2 "NEWblack:D_DO-35_SOD27_P7.62mm_Horizontal" V 6100 2400 50  0001 C CNN
 F 3 "~" V 6100 2400 50  0001 C CNN
 	1    6100 2400
@@
 F 0 "D6" V 6846 2330 50  0000 R CNN
 F 1 "D_Small" V 6755 2330 50  0000 R CNN
-F 2 "Diode_THT:D_DO-35_SOD27_P7.62mm_Horizontal" V 6800 2400 50  0001 C CNN
+F 2 "NEWblack:D_DO-35_SOD27_P7.62mm_Horizontal" V 6800 2400 50  0001 C CNN
 F 3 "~" V 6800 2400 50  0001 C CNN
 	1    6800 2400
@@
 F 0 "D7" V 7346 2330 50  0000 R CNN
 F 1 "D_Small" V 7255 2330 50  0000 R CNN
-F 2 "Diode_THT:D_DO-35_SOD27_P7.62mm_Horizontal" V 7300 2400 50  0001 C CNN
+F 2 "NEWblack:D_DO-35_SOD27_P7.62mm_Horizontal" V 7300 2400 50  0001 C CNN
 F 3 "~" V 7300 2400 50  0001 C CNN
 	1    7300 2400
@@
 F 0 "D8" V 7796 2330 50  0000 R CNN
 F 1 "D_Small" V 7705 2330 50  0000 R CNN
-F 2 "Diode_THT:D_DO-35_SOD27_P7.62mm_Horizontal" V 7750 2400 50  0001 C CNN
+F 2 "NEWblack:D_DO-35_SOD27_P7.62mm_Horizontal" V 7750 2400 50  0001 C CNN
 F 3 "~" V 7750 2400 50  0001 C CNN
 	1    7750 2400
@@
 F 0 "D10" V 6146 3130 50  0000 R CNN
 F 1 "D_Small" V 6055 3130 50  0000 R CNN
-F 2 "Diode_THT:D_DO-35_SOD27_P7.62mm_Horizontal" V 6100 3200 50  0001 C CNN
+F 2 "NEWblack:D_DO-35_SOD27_P7.62mm_Horizontal" V 6100 3200 50  0001 C CNN
 F 3 "~" V 6100 3200 50  0001 C CNN
 	1    6100 3200
@@
 F 0 "D11" V 6846 3130 50  0000 R CNN
 F 1 "D_Small" V 6755 3130 50  0000 R CNN
-F 2 "Diode_THT:D_DO-35_SOD27_P7.62mm_Horizontal" V 6800 3200 50  0001 C CNN
+F 2 "NEWblack:D_DO-35_SOD27_P7.62mm_Horizontal" V 6800 3200 50  0001 C CNN
 F 3 "~" V 6800 3200 50  0001 C CNN
 	1    6800 3200
@@
 F 0 "D12" V 7346 3130 50  0000 R CNN
 F 1 "D_Small" V 7255 3130 50  0000 R CNN
-F 2 "Diode_THT:D_DO-35_SOD27_P7.62mm_Horizontal" V 7300 3200 50  0001 C CNN
+F 2 "NEWblack:D_DO-35_SOD27_P7.62mm_Horizontal" V 7300 3200 50  0001 C CNN
 F 3 "~" V 7300 3200 50  0001 C CNN
 	1    7300 3200
@@
 F 0 "D13" V 7796 3130 50  0000 R CNN
 F 1 "D_Small" V 7705 3130 50  0000 R CNN
-F 2 "Diode_THT:D_DO-35_SOD27_P7.62mm_Horizontal" V 7750 3200 50  0001 C CNN
+F 2 "NEWblack:D_DO-35_SOD27_P7.62mm_Horizontal" V 7750 3200 50  0001 C CNN
 F 3 "~" V 7750 3200 50  0001 C CNN
 	1    7750 3200
@@
 F 0 "D15" V 6146 3830 50  0000 R CNN
 F 1 "D_Small" V 6055 3830 50  0000 R CNN
-F 2 "Diode_THT:D_DO-35_SOD27_P7.62mm_Horizontal" V 6100 3900 50  0001 C CNN
+F 2 "NEWblack:D_DO-35_SOD27_P7.62mm_Horizontal" V 6100 3900 50  0001 C CNN
 F 3 "~" V 6100 3900 50  0001 C CNN
 	1    6100 3900
@@
 F 0 "D16" V 6846 3830 50  0000 R CNN
 F 1 "D_Small" V 6755 3830 50  0000 R CNN
-F 2 "Diode_THT:D_DO-35_SOD27_P7.62mm_Horizontal" V 6800 3900 50  0001 C CNN
+F 2 "NEWblack:D_DO-35_SOD27_P7.62mm_Horizontal" V 6800 3900 50  0001 C CNN
 F 3 "~" V 6800 3900 50  0001 C CNN
 	1    6800 3900
@@
 F 0 "D17" V 7346 3830 50  0000 R CNN
 F 1 "D_Small" V 7255 3830 50  0000 R CNN
-F 2 "Diode_THT:D_DO-35_SOD27_P7.62mm_Horizontal" V 7300 3900 50  0001 C CNN
+F 2 "NEWblack:D_DO-35_SOD27_P7.62mm_Horizontal" V 7300 3900 50  0001 C CNN
 F 3 "~" V 7300 3900 50  0001 C CNN
 	1    7300 3900
@@
 F 0 "D18" V 7796 3830 50  0000 R CNN
 F 1 "D_Small" V 7705 3830 50  0000 R CNN
-F 2 "Diode_THT:D_DO-35_SOD27_P7.62mm_Horizontal" V 7750 3900 50  0001 C CNN
+F 2 "NEWblack:D_DO-35_SOD27_P7.62mm_Horizontal" V 7750 3900 50  0001 C CNN
 F 3 "~" V 7750 3900 50  0001 C CNN
 	1    7750 3900
@@
 F 0 "D19" V 6146 4530 50  0000 R CNN
 F 1 "D_Small" V 6055 4530 50  0000 R CNN
-F 2 "Diode_THT:D_DO-35_SOD27_P7.62mm_Horizontal" V 6100 4600 50  0001 C CNN
+F 2 "NEWblack:D_DO-35_SOD27_P7.62mm_Horizontal" V 6100 4600 50  0001 C CNN
 F 3 "~" V 6100 4600 50  0001 C CNN
 	1    6100 4600
@@
 F 0 "D20" V 6846 4530 50  0000 R CNN
 F 1 "D_Small" V 6755 4530 50  0000 R CNN
-F 2 "Diode_THT:D_DO-35_SOD27_P7.62mm_Horizontal" V 6800 4600 50  0001 C CNN
+F 2 "NEWblack:D_DO-35_SOD27_P7.62mm_Horizontal" V 6800 4600 50  0001 C CNN
 F 3 "~" V 6800 4600 50  0001 C CNN
 	1    6800 4600
@@
 F 0 "D21" V 7346 4530 50  0000 R CNN
 F 1 "D_Small" V 7255 4530 50  0000 R CNN
-F 2 "Diode_THT:D_DO-35_SOD27_P7.62mm_Horizontal" V 7300 4600 50  0001 C CNN
+F 2 "NEWblack:D_DO-35_SOD27_P7.62mm_Horizontal" V 7300 4600 50  0001 C CNN
 F 3 "~" V 7300 4600 50  0001 C CNN
 	1    7300 4600
@@
 F 0 "D22" V 7796 4530 50  0000 R CNN
 F 1 "D_Small" V 7705 4530 50  0000 R CNN
-F 2 "Diode_THT:D_DO-35_SOD27_P7.62mm_Horizontal" V 7750 4600 50  0001 C CNN
+F 2 "NEWblack:D_DO-35_SOD27_P7.62mm_Horizontal" V 7750 4600 50  0001 C CNN
 F 3 "~" V 7750 4600 50  0001 C CNN
 	1    7750 4600
@@
 F 0 "D23" V 8746 4530 50  0000 R CNN
 F 1 "D_Small" V 8655 4530 50  0000 R CNN
-F 2 "Diode_THT:D_DO-35_SOD27_P7.62mm_Horizontal" V 8700 4600 50  0001 C CNN
+F 2 "NEWblack:D_DO-35_SOD27_P7.62mm_Horizontal" V 8700 4600 50  0001 C CNN
 F 3 "~" V 8700 4600 50  0001 C CNN
 	1    8700 4600
@@
 F 0 "D14" V 8746 3780 50  0000 R CNN
 F 1 "D_Small" V 8655 3780 50  0000 R CNN
-F 2 "Diode_THT:D_DO-35_SOD27_P7.62mm_Horizontal" V 8700 3850 50  0001 C CNN
+F 2 "NEWblack:D_DO-35_SOD27_P7.62mm_Horizontal" V 8700 3850 50  0001 C CNN
 F 3 "~" V 8700 3850 50  0001 C CNN
 	1    8700 3850
@@
 P 4600 5250
 F 0 "SW3" H 4600 5535 50  0000 C CNN
-F 1 "SW_Push" H 4600 5444 50  0000 C CNN
+F 1 "RESET" H 4600 5444 50  0000 C CNN
 F 2 "random-keyboard-parts:PushButton_6x6mm_TH" H 4600 5450 50  0001 C CNN
 F 3 "~" H 4600 5450 50  0001 C CNN
@@
 F 0 "D9" V 9196 3080 50  0000 R CNN
 F 1 "D_Small" V 9105 3080 50  0000 R CNN
-F 2 "Diode_THT:D_DO-35_SOD27_P7.62mm_Horizontal" V 9150 3150 50  0001 C CNN
+F 2 "NEWblack:D_DO-35_SOD27_P7.62mm_Horizontal" V 9150 3150 50  0001 C CNN
 F 3 "~" V 9150 3150 50  0001 C CNN
 	1    9150 3150

Commit message: Updated pcb and plate designs, added led difusion layer to chasis
Connections:
- net D2: no longer SW2.A
- net F5: now also SW2.A
Changed lines of the file:
@@
 Text GLabel 9700 4300 2    50   Input ~ 0
 RE_B2
-Text GLabel 9700 4500 2    50   Input ~ 0
-RE_A2
 Wire Wire Line
 	9550 4500 9700 4500
@@
 Wire Wire Line
 	1700 1700 1900 1700
-Text GLabel 6050 6250 2    50   Input ~ 0
-D2
 Text GLabel 5800 5950 0    50   Input ~ 0
 RE_B1
@@
 Text GLabel 5800 6150 0    50   Input ~ 0
 RE_B2
-Text GLabel 5800 6250 0    50   Input ~ 0
-RE_A2
-Wire Wire Line
-	5800 6250 6050 6250
 Wire Wire Line
 	5800 6150 6050 6150
@@
 	1    0    0    -1
 $EndComp
+Text GLabel 9700 4500 2    50   Input ~ 0
+RE_A1
 $EndSCHEMATC
